Commit message: 找到了好多东西，女人

File: learning/C++/ros2/urdfLearning/urdf/third_robot.urdf (robot description, URDF)
Before this commit: robot third_robot, 10 links, 9 joints
Links:
- link base_link: mass None -> 1.0; geometry collision box size=0.2 0.2 0.12; visual box size=0.2 0.2 0.12
- link camera01_link: mass None -> 0.5; geometry collision box size=0.04 0.04 0.04; visual box size=0.04 0.04 0.04
- link camera02_link: mass None -> 0.5; geometry collision box size=0.04 0.04 0.04; visual box size=0.04 0.04 0.04
- link laser: mass None -> 0.5; geometry collision cylinder length=0.02 radius=0.02; visual cylinder length=0.02 radius=0.02
- link laser_link: mass None -> 0.5; geometry collision cylinder length=0.10 radius=0.01; visual cylinder length=0.10 radius=0.01
- link wheel01_link: mass None -> 0.5; geometry collision cylinder length=0.04 radius=0.04; visual cylinder length=0.04 radius=0.04
- link wheel02_link: mass None -> 0.5; geometry collision cylinder length=0.04 radius=0.04; visual cylinder length=0.04 radius=0.04
- link wheel03_link: mass None -> 0.5; geometry collision cylinder length=0.04 radius=0.04; visual cylinder length=0.04 radius=0.04
- link wheel04_link: mass None -> 0.5; geometry collision cylinder length=0.04 radius=0.04; visual cylinder length=0.04 radius=0.04

File: learning/C++/ros2/urdfLearning/urdf/third_robot/base.urdf.xacro (robot description, xacro)
@@ -1,4 +1,5 @@
 <?xml version="1.0"?>
 <robot xmlns:xacro="http://www.ros.org/wiki/xacro">
+<xacro:include filename="$(find cpp_demo)/urdf/inertial.xacro"/>
     <xacro:macro name="base_link" params="xyz">
         <link name="base_shadow">
@@ -14,4 +15,14 @@
                 </material>
             </visual>
+            <collision>
+            <origin xyz="0.0 0.0 0.0" rpy="0.0 0.0 0.0"/>
+                <geometry>
+                    <box size="${xyz}"/>
+                </geometry>
+                <material name="white">
+                    <color rgba="1.0 1.0 1.0 0.5"/>
+                </material>
+            </collision>
+            <xacro:box_inertia m="1.0" w="0.2" h="0.2" d="0.12"/>
         </link>
         <joint name="base_joint" type="fixed">

File: learning/C++/ros2/urdfLearning/urdf/third_robot/camera.urdf.xacro (robot description, xacro)
@@ -1,4 +1,5 @@
 <?xml version="1.0"?>
 <robot xmlns:xacro="http://www.ros.org/wiki/xacro">
+<xacro:include filename="$(find cpp_demo)/urdf/inertial.xacro"/>
     <xacro:macro name="camera_link" params="camera_name xyz">
         <link name="${camera_name}_link">
@@ -12,4 +13,14 @@
                 </material>
             </visual>
+            <collision>
+                <origin xyz="0.0 0.0 0.0" rpy="0.0 0.0 0.0"/>
+                    <geometry>
+                        <box size="0.04 0.04 0.04"/>
+                    </geometry>
+                    <material name="black">
+                        <color rgba="0.0 0.0 0.0 0.5"/>
+                    </material>
+            </collision>
+            <xacro:box_inertia m="0.5" w="0.04" d="0.04" h="0.04" />
         </link>
         <joint name="${camera_name}_joint" type="fixed">

File: learning/C++/ros2/urdfLearning/urdf/third_robot/laser.urdf.xacro (robot description, xacro)
@@ -1,4 +1,5 @@
 <?xml version="1.0"?>
 <robot xmlns:xacro="http://www.ros.org/wiki/xacro">
+<xacro:include filename="$(find cpp_demo)/urdf/inertial.xacro"/>
     <xacro:macro name="laser_link" params="xyz">
         <link name="laser_link">
@@ -12,4 +13,14 @@
                 </material>
             </visual>
+            <collision>
+                <origin xyz="${xyz}" rpy="0.0 0.0 0.0"/>
+                <geometry>
+                    <cylinder radius="0.01" length="0.10"/>
+                </geometry>
+                <material name="black">
+                    <color rgba="0.0 0.0 0.0 0.5"/>
+                </material>
+            </collision>
+            <xacro:cylinder_inertia m="0.5" r="0.01" h="0.10" />
         </link>
         <link name="laser">
@@ -23,4 +34,14 @@
                 </material>
             </visual>
+            <collision>
+                <origin xyz="${xyz}" rpy="0.0 0.0 0.0"/>
+                <geometry>
+                    <cylinder radius="0.02" length="0.02"/>
+                </geometry>
+                <material name="black">
+                    <color rgba="0.0 0.0 0.0 0.5"/>
+                </material>
+            </collision>
+            <xacro:cylinder_inertia m="0.5" r="0.02" h="0.02" />
         </link>
         <joint name="laser_joint" type="fixed">

File: learning/C++/ros2/urdfLearning/urdf/third_robot/wheel.urdf.xacro (robot description, xacro)
@@ -12,4 +12,14 @@
                 </material>
             </visual>
+            <collision>
+                <origin xyz="0.0 0.0 0.0" rpy="1.5708 0.0 0.0"/>
+                    <geometry>
+                        <cylinder length="0.04" radius="0.04"/>
+                    </geometry>
+                    <material name="black">
+                        <color rgba="0.0 0.0 0.0 0.5"/>
+                    </material>
+            </collision>
+            <xacro:cylinder_inertia m="0.5" r="0.04" h="0.04" />
         </link>
         <joint name="${wheel_name}_joint" type="fixed">

Commit message: 吸取教训了，记得备份

File: learning/C++/ros2/urdfLearning/urdf/third_robot.urdf (robot description, URDF)
Before this commit: robot third_robot, 10 links, 9 joints
Joints:
- joint wheel01_joint: axis (none) -> 0 1 0; limit (none) -> effort=20.0 velocity=10.0; type fixed -> continuous
- joint wheel02_joint: axis (none) -> 0 1 0; limit (none) -> effort=20.0 velocity=10.0; type fixed -> continuous
- joint wheel03_joint: axis (none) -> 0 1 0; limit (none) -> effort=0.0 velocity=10.0; type fixed -> continuous
- joint wheel04_joint: axis (none) -> 0 1 0; limit (none) -> effort=0.0 velocity=10.0; type fixed -> continuous

File: learning/C++/ros2/urdfLearning/urdf/third_robot.xacro (robot description, xacro)
@@ -1,15 +1,21 @@
 <?xml version="1.0"?>
 <robot xmlns:xacro="http://www.ros.org/wiki/xacro" name="third_robot">
-<xacro:include filename="$(find cpp_demo)/urdf/third_robot/base.urdf.xacro"/>
-<xacro:include filename="$(find cpp_demo)/urdf/third_robot/camera.urdf.xacro"/>
-<xacro:include filename="$(find cpp_demo)/urdf/third_robot/laser.urdf.xacro"/>
-<xacro:include filename="$(find cpp_demo)/urdf/third_robot/wheel.urdf.xacro"/>
-<xacro:base_link xyz="0.2 0.2 0.12"/>
-<xacro:camera_link camera_name="camera01" xyz="0.04 -0.04 0.08"/>
-<xacro:camera_link camera_name="camera02" xyz="0.04 0.04 0.08"/>
-<xacro:laser_link xyz="0.0 0.0 0.05"/>
-<xacro:wheel_link wheel_name="wheel01" xyz="0.05 0.1 -0.06"/>
-<xacro:wheel_link wheel_name="wheel02" xyz="0.05 -0.1 -0.06"/>
-<xacro:wheel_link wheel_name="wheel03" xyz="-0.05 0.1 -0.06"/>
-<xacro:wheel_link wheel_name="wheel04" xyz="-0.05 -0.1 -0.06"/>
+  <xacro:include filename="$(find cpp_demo)/urdf/third_robot/base.urdf.xacro"/>
+  <xacro:include filename="$(find cpp_demo)/urdf/third_robot/camera.urdf.xacro"/>
+  <xacro:include filename="$(find cpp_demo)/urdf/third_robot/laser.urdf.xacro"/>
+  <xacro:include filename="$(find cpp_demo)/urdf/third_robot/wheel.urdf.xacro"/>
+  <xacro:include filename="$(find cpp_demo)/urdf/diff_drive_plugin.xacro"/>
+  <!-- 底盘 0.2(x) 0.2(y) 0.12(z) -->
+  <xacro:base_link xyz="0.2 0.2 0.12"/>
+  <xacro:camera_link camera_name="camera01" xyz="0.04 -0.04 0.08"/>
+  <xacro:camera_link camera_name="camera02" xyz="0.04 0.04 0.08"/>
+  <xacro:laser_link xyz="0.0 0.0 0.05"/>
+  <!-- 驱动轮 -->
+  <xacro:drive_wheel wheel_name="wheel01" xyz="0.05 0.1 -0.06"/>
+  <xacro:drive_wheel wheel_name="wheel02" xyz="0.05 -0.1 -0.06"/>
+  <!-- 随动轮 -->
+  <xacro:passive_wheel wheel_name="wheel03" xyz="-0.05 0.1 -0.06"/>
+  <xacro:passive_wheel wheel_name="wheel04" xyz="-0.05 -0.1 -0.06"/>
+  <!-- 加载差速插件 -->
+  <xacro:diff_drive_plugin/>
 </robot>

File: learning/C++/ros2/urdfLearning/urdf/third_robot/laser.urdf.xacro (robot description, xacro)
@@ -31,5 +31,5 @@
                 </geometry>
                 <material name="black">
-                    <color rgba="0.0 0.0 0.0 0.5"/>
+                    <color rgba="0.0 0.0 0.0 1.0"/>
                 </material>
             </visual>
@@ -40,5 +40,5 @@
                 </geometry>
                 <material name="black">
-                    <color rgba="0.0 0.0 0.0 0.5"/>
+                    <color rgba="0.0 0.0 0.0 1.0"/>
                 </material>
             </collision>

File: learning/C++/ros2/urdfLearning/urdf/third_robot/wheel.urdf.xacro (robot description, xacro)
@@ -1,31 +1,85 @@
 <?xml version="1.0"?>
 <robot xmlns:xacro="http://www.ros.org/wiki/xacro">
-    <xacro:macro name="wheel_link" params="wheel_name xyz">
-        <link name="${wheel_name}_link">
-            <visual>
-                <origin xyz="0.0 0.0 0.0" rpy="1.5708 0.0 0.0"/>
-                <geometry>
-                    <cylinder length="0.04" radius="0.04"/>
-                </geometry>
-                <material name="black">
-                    <color rgba="0.0 0.0 0.0 0.5"/>
-                </material>
-            </visual>
-            <collision>
-                <origin xyz="0.0 0.0 0.0" rpy="1.5708 0.0 0.0"/>
-                    <geometry>
-                        <cylinder length="0.04" radius="0.04"/>
-                    </geometry>
-                    <material name="black">
-                        <color rgba="0.0 0.0 0.0 0.5"/>
-                    </material>
-            </collision>
-            <xacro:cylinder_inertia m="0.5" r="0.04" h="0.04" />
-        </link>
-        <joint name="${wheel_name}_joint" type="fixed">
-            <parent link="base_link"/>
-            <child link="${wheel_name}_link"/>
-            <origin xyz="${xyz}" rpy="0.0 0.0 0.0"/>
-        </joint>
-    </xacro:macro>
+  <!-- 轮子专用圆柱惯性宏（勿与 inertial.xacro 里的 cylinder_inertia 重名）-->
+  <!-- 圆柱几何轴沿Y（visual/collision已旋转90°），关节axis=0 1 0，即绕Y旋转 -->
+  <xacro:macro name="wheel_cylinder_inertia" params="m r h">
+    <inertial>
+      <mass value="${m}"/>
+      <inertia
+        ixx="${m*(3*r*r + h*h)/12}"
+        ixy="0.0"
+        ixz="0.0"
+        iyy="${0.5*m*r*r}"
+        izz="${m*(3*r*r + h*h)/12}"
+        iyz="0.0"
+      />
+    </inertial>
+  </xacro:macro>
+  <!-- 驱动轮：revolute 差速控制，摩擦大保证抓地 -->
+  <xacro:macro name="drive_wheel" params="wheel_name xyz">
+    <link name="${wheel_name}_link">
+      <visual>
+        <origin xyz="0.0 0.0 0.0" rpy="1.5708 0.0 0.0"/>
+        <geometry>
+          <cylinder length="0.04" radius="0.04"/>
+        </geometry>
+        <material name="black">
+          <color rgba="0.0 0.0 0.0 1.0"/>
+        </material>
+      </visual>
+      <collision>
+        <origin xyz="0.0 0.0 0.0" rpy="1.5708 0.0 0.0"/>
+        <geometry>
+          <cylinder length="0.04" radius="0.04"/>
+        </geometry>
+      </collision>
+      <xacro:wheel_cylinder_inertia m="0.5" r="0.04" h="0.04" />
+    </link>
+    <!-- continuous：轮子必须用连续旋转。revolute不写lower/upper默认0~0，轮子会被锁死 -->
+    <joint name="${wheel_name}_joint" type="continuous">
+      <parent link="base_link"/>
+      <child link="${wheel_name}_link"/>
+      <origin xyz="${xyz}" rpy="0.0 0.0 0.0"/>
+      <!-- 圆柱轴沿Y，必须显式指定转轴；正向速度=前进(+X) -->
+      <axis xyz="0 1 0"/>
+      <limit effort="20.0" velocity="10.0"/>
+    </joint>
+    <gazebo reference="${wheel_name}_link">
+      <mu1>1.0</mu1>
+      <mu2>1.0</mu2>
+    </gazebo>
+  </xacro:macro>
+  <!-- 随动轮：自由旋转revolute，effort=0无驱动力 -->
+  <!-- 摩擦调低：4轮均为平行Y轴轮，转向靠横向打滑，摩擦太大会转不动 -->
+  <xacro:macro name="passive_wheel" params="wheel_name xyz">
+    <link name="${wheel_name}_link">
+      <visual>
+        <origin xyz="0.0 0.0 0.0" rpy="1.5708 0.0 0.0"/>
+        <geometry>
+          <cylinder length="0.04" radius="0.04"/>
+        </geometry>
+        <material name="black">
+          <color rgba="0.0 0.0 0.0 1.0"/>
+        </material>
+      </visual>
+      <collision>
+        <origin xyz="0.0 0.0 0.0" rpy="1.5708 0.0 0.0"/>
+        <geometry>
+          <cylinder length="0.04" radius="0.04"/>
+        </geometry>
+      </collision>
+      <xacro:wheel_cylinder_inertia m="0.5" r="0.04" h="0.04" />
+    </link>
+    <joint name="${wheel_name}_joint" type="continuous">
+      <parent link="base_link"/>
+      <child link="${wheel_name}_link"/>
+      <origin xyz="${xyz}" rpy="0.0 0.0 0.0"/>
+      <axis xyz="0 1 0"/>
+      <limit effort="0.0" velocity="10.0"/>
+    </joint>
+    <gazebo reference="${wheel_name}_link">
+      <mu1>0.3</mu1>
+      <mu2>0.3</mu2>
+    </gazebo>
+  </xacro:macro>
 </robot>
