Commit message: 赶快提交一下，又修好了

File: learning/C++/ros2/daohangLearning/urdf/diff_drive_plugin.xacro (robot description, xacro)
@@ -19,5 +19,6 @@
         <tf_topic>/tf</tf_topic>
         <frame_id>odom</frame_id>
-        <child_frame_id>base_link</child_frame_id>
+        <!-- 差速里程计积分的是轮轴中点在地面上的投影点，即 base_footprint -->
+        <child_frame_id>base_footprint</child_frame_id>
       </plugin>
     </gazebo>

File: learning/C++/ros2/daohangLearning/urdf/robot.urdf (robot description, URDF)
Before this commit: robot robot, 10 links, 9 joints
Links:
- added link base_footprint
Joints:
- added joint base_footprint_joint: type fixed, parent base_footprint, child base_link, origin xyz=0.0 0.0 0.10 rpy=0.0 0.0 0.0

File: learning/C++/ros2/daohangLearning/urdf/robot/base.urdf.xacro (robot description, xacro)
@@ -3,4 +3,15 @@
 <xacro:include filename="$(find cpp_demo)/urdf/inertial.xacro"/>
     <xacro:macro name="base_link" params="xyz">
+        <!-- 根link：无惯性的 dummy link。
+             kdl_parser 要求根 link 不能带惯性，否则 robot_state_publisher
+             每次启动都会告警；base_footprint 同时也是轮子接地点的投影，
+             与差速插件 odom->base_footprint 的 TF 数值严格一致 -->
+        <link name="base_footprint"/>
+        <joint name="base_footprint_joint" type="fixed">
+            <parent link="base_footprint"/>
+            <child link="base_link"/>
+            <!-- 轮轴中心在 base_link 下方 0.06，轮半径 0.04，接地点即 -0.10 -->
+            <origin xyz="0.0 0.0 0.10" rpy="0.0 0.0 0.0"/>
+        </joint>
         <link name="base_shadow">
         </link>
